Commit message: added front right wheel on urdf

File: src/uav_description/urdf/pioneer.urdf (robot description, URDF)
Before this commit: robot pioneer3at_body, 9 links, 8 joints
Links:
- added link p3at_front_right_axle, mass 0.1; collision box size=0.01 0.01 0.01; visual mesh filename=../meshes/p3at_meshes/axle.dae
- added link p3at_front_right_hub, mass 0.1; collision box size=0.01 0.01 0.01; visual mesh filename=../meshes/p3at_meshes/right_hubcap.dae
- added link p3at_front_right_wheel, mass 0.5; collision mesh filename=../meshes/p3at_meshes/wheel.dae; visual mesh filename=../meshes/p3at_meshes/wheel.dae
Joints:
- added joint base_front_right_axle_joint: type fixed, parent base_link, child p3at_front_right_axle, origin xyz=0.135 -0.156 0.111 rpy=0 0 0
- added joint base_front_right_hub_joint: type fixed, parent p3at_front_right_axle, child p3at_front_right_hub, origin xyz=0 -0.041 0 rpy=0 0 0
- added joint p3at_front_right_wheel_joint: type continuous, parent p3at_front_right_hub, child p3at_front_right_wheel, origin xyz=0 0 0 rpy=0 0 0, axis 0 1 0, limit effort=100 velocity=100

Commit message: added all wheels to urdf

File: src/uav_description/urdf/pioneer.urdf (robot description, URDF)
Before this commit: robot pioneer3at_body, 12 links, 11 joints
Links:
- added link p3at_back_left_axle, mass 0.1; collision box size=0.01 0.01 0.01; visual mesh filename=../meshes/p3at_meshes/axle.dae
- added link p3at_back_left_hub, mass 0.1; collision box size=0.01 0.01 0.01; visual mesh filename=../meshes/p3at_meshes/left_hubcap.dae
- added link p3at_back_left_wheel, mass 0.5; collision mesh filename=../meshes/p3at_meshes/wheel.dae; visual mesh filename=../meshes/p3at_meshes/wheel.dae
- added link p3at_back_right_axle, mass 0.1; collision box size=0.01 0.01 0.01; visual mesh filename=../meshes/p3at_meshes/axle.dae
- added link p3at_back_right_hub, mass 0.1; collision box size=0.01 0.01 0.01; visual mesh filename=../meshes/p3at_meshes/right_hubcap.dae
- added link p3at_back_right_wheel, mass 0.5; collision mesh filename=../meshes/p3at_meshes/wheel.dae; visual mesh filename=../meshes/p3at_meshes/wheel.dae
Joints:
- added joint base_back_left_axle_joint: type fixed, parent base_link, child p3at_back_left_axle, origin xyz=-0.135 0.156 0.111 rpy=0 0 0
- added joint base_back_left_hub_joint: type fixed, parent p3at_back_left_axle, child p3at_back_left_hub, origin xyz=0 0.041 0 rpy=0 0 0
- added joint base_back_right_axle_joint: type fixed, parent base_link, child p3at_back_right_axle, origin xyz=-0.135 -0.156 0.111 rpy=0 0 0
- added joint base_back_right_hub_joint: type fixed, parent p3at_back_right_axle, child p3at_back_right_hub, origin xyz=0 -0.041 0 rpy=0 0 0
- added joint p3at_back_left_wheel_joint: type continuous, parent p3at_back_left_hub, child p3at_back_left_wheel, origin xyz=0 0 0 rpy=0 0 0, axis 0 1 0, limit effort=100 velocity=100
- added joint p3at_back_right_wheel_joint: type continuous, parent p3at_back_right_hub, child p3at_back_right_wheel, origin xyz=0 0 0 rpy=0 0 0, axis 0 1 0, limit effort=100 velocity=100
