Commit message: updates

File: src/uav_sim/models/urdf/pioneer.urdf (robot description, URDF)
Before this commit: robot pioneer3at_body, 18 links, 17 joints
Links:
- link chassis: geometry collision mesh filename=package://uav_sim/models/meshes/chassis.dae; visual mesh filename=package://uav_sim/models/meshes/chassis.dae
- link laser_frame: geometry collision box size=0.01 0.01 0.01; visual mesh filename=package://uav_sim/models/meshes/hokuyo1.dae
- link p3at_back_left_axle: geometry collision box size=0.01 0.01 0.01; visual mesh filename=package://uav_sim/models/meshes/p3at_meshes/axle.dae
- link p3at_back_left_hub: geometry collision box size=0.01 0.01 0.01; visual mesh filename=package://uav_sim/models/meshes/p3at_meshes/left_hubcap.dae
- link p3at_back_left_wheel: geometry collision mesh filename=package://uav_sim/models/meshes/p3at_meshes/wheel.dae; visual mesh filename=package://uav_sim/models/meshes/p3at_meshes/wheel.dae
- link p3at_back_right_axle: geometry collision box size=0.01 0.01 0.01; visual mesh filename=package://uav_sim/models/meshes/p3at_meshes/axle.dae
- link p3at_back_right_hub: geometry collision box size=0.01 0.01 0.01; visual mesh filename=package://uav_sim/models/meshes/p3at_meshes/right_hubcap.dae
- link p3at_back_right_wheel: geometry collision mesh filename=package://uav_sim/models/meshes/p3at_meshes/wheel.dae; visual mesh filename=package://uav_sim/models/meshes/p3at_meshes/wheel.dae
- link p3at_front_left_axle: geometry collision box size=0.01 0.01 0.01; visual mesh filename=package://uav_sim/models/meshes/p3at_meshes/axle.dae
- link p3at_front_left_hub: geometry collision box size=0.01 0.01 0.01; visual mesh filename=package://uav_sim/models/meshes/p3at_meshes/left_hubcap.dae
- link p3at_front_left_wheel: geometry collision mesh filename=package://uav_sim/models/meshes/p3at_meshes/wheel.dae; visual mesh filename=package://uav_sim/models/meshes/p3at_meshes/wheel.dae
- link p3at_front_right_axle: geometry collision box size=0.01 0.01 0.01; visual mesh filename=package://uav_sim/models/meshes/p3at_meshes/axle.dae
- link p3at_front_right_hub: geometry collision box size=0.01 0.01 0.01; visual mesh filename=package://uav_sim/models/meshes/p3at_meshes/right_hubcap.dae
- link p3at_front_right_wheel: geometry collision mesh filename=package://uav_sim/models/meshes/p3at_meshes/wheel.dae; visual mesh filename=package://uav_sim/models/meshes/p3at_meshes/wheel.dae
- link top_plate: geometry collision box size=0.1 0.1 0.1; visual mesh filename=package://uav_sim/models/meshes/top.dae
