Commit message: updates

File: src/uav_sim/models/pioneer.urdf (robot description, URDF)
Before this commit: robot pioneer3at_body, 18 links, 17 joints
Links:
- link chassis: geometry collision mesh filename=package://chassis.dae; visual mesh filename=package://chassis.dae
- link laser_frame: geometry collision box size=0.01 0.01 0.01; visual mesh filename=package://hokuyo1.dae
- link p3at_back_left_axle: geometry collision box size=0.01 0.01 0.01; visual mesh filename=package://p3at_meshes/axle.dae
- link p3at_back_left_hub: geometry collision box size=0.01 0.01 0.01; visual mesh filename=package://p3at_meshes/left_hubcap.dae
- link p3at_back_left_wheel: geometry collision mesh filename=package://p3at_meshes/wheel.dae; visual mesh filename=package://p3at_meshes/wheel.dae
- link p3at_back_right_axle: geometry collision box size=0.01 0.01 0.01; visual mesh filename=package://p3at_meshes/axle.dae
- link p3at_back_right_hub: geometry collision box size=0.01 0.01 0.01; visual mesh filename=package://p3at_meshes/right_hubcap.dae
- link p3at_back_right_wheel: geometry collision mesh filename=package://p3at_meshes/wheel.dae; visual mesh filename=package://p3at_meshes/wheel.dae
- link p3at_front_left_axle: geometry collision box size=0.01 0.01 0.01; visual mesh filename=package://p3at_meshes/axle.dae
- link p3at_front_left_hub: geometry collision box size=0.01 0.01 0.01; visual mesh filename=package://p3at_meshes/left_hubcap.dae
- link p3at_front_left_wheel: geometry collision mesh filename=package://p3at_meshes/wheel.dae; visual mesh filename=package://p3at_meshes/wheel.dae
- link p3at_front_right_axle: geometry collision box size=0.01 0.01 0.01; visual mesh filename=package://p3at_meshes/axle.dae
- link p3at_front_right_hub: geometry collision box size=0.01 0.01 0.01; visual mesh filename=package://p3at_meshes/right_hubcap.dae
- link p3at_front_right_wheel: geometry collision mesh filename=package://p3at_meshes/wheel.dae; visual mesh filename=package://p3at_meshes/wheel.dae
- link top_plate: geometry collision box size=0.1 0.1 0.1; visual mesh filename=package://top.dae

Commit message: updated paths to render pioneer in both gazebo and rviz (partial)

File: src/uav_sim/models/pioneer.urdf (robot description, URDF)
Before this commit: robot pioneer3at_body, 18 links, 17 joints
Links:
- link chassis: geometry collision mesh filename=package://uav_sim/meshes/chassis.dae; visual mesh filename=package://uav_sim/meshes/chassis.dae
- link laser_frame: geometry collision box size=0.01 0.01 0.01; visual mesh filename=package://uav_sim/meshes/hokuyo1.dae
- link p3at_back_left_axle: geometry collision box size=0.01 0.01 0.01; visual mesh filename=package://uav_sim/meshes/p3at_meshes/axle.dae
- link p3at_back_left_hub: geometry collision box size=0.01 0.01 0.01; visual mesh filename=package://uav_sim/meshes/p3at_meshes/left_hubcap.dae
- link p3at_back_left_wheel: geometry collision mesh filename=package://uav_sim/meshes/p3at_meshes/wheel.dae; visual mesh filename=package://uav_sim/meshes/p3at_meshes/wheel.dae
- link p3at_back_right_axle: geometry collision box size=0.01 0.01 0.01; visual mesh filename=package://uav_sim/meshes/p3at_meshes/axle.dae
- link p3at_back_right_hub: geometry collision box size=0.01 0.01 0.01; visual mesh filename=package://uav_sim/meshes/p3at_meshes/right_hubcap.dae
- link p3at_back_right_wheel: geometry collision mesh filename=package://uav_sim/meshes/p3at_meshes/wheel.dae; visual mesh filename=package://uav_sim/meshes/p3at_meshes/wheel.dae
- link p3at_front_left_axle: geometry collision box size=0.01 0.01 0.01; visual mesh filename=package://uav_sim/meshes/p3at_meshes/axle.dae
- link p3at_front_left_hub: geometry collision box size=0.01 0.01 0.01; visual mesh filename=package://uav_sim/meshes/p3at_meshes/left_hubcap.dae
- link p3at_front_left_wheel: geometry collision mesh filename=package://uav_sim/meshes/p3at_meshes/wheel.dae; visual mesh filename=package://uav_sim/meshes/p3at_meshes/wheel.dae
- link p3at_front_right_axle: geometry collision box size=0.01 0.01 0.01; visual mesh filename=package://uav_sim/meshes/p3at_meshes/axle.dae
- link p3at_front_right_hub: geometry collision box size=0.01 0.01 0.01; visual mesh filename=package://uav_sim/meshes/p3at_meshes/right_hubcap.dae
- link p3at_front_right_wheel: geometry collision mesh filename=package://uav_sim/meshes/p3at_meshes/wheel.dae; visual mesh filename=package://uav_sim/meshes/p3at_meshes/wheel.dae
- link top_plate: geometry collision box size=0.1 0.1 0.1; visual mesh filename=package://uav_sim/meshes/top.dae

Commit message: update launch file to include additional joint state and pose parameters; modify URDF for correct joint parent links

File: src/uav_sim/models/pioneer.urdf (robot description, URDF)
Before this commit: robot pioneer3at_body, 18 links, 17 joints
Joints:
- joint base_back_left_axle_joint: origin xyz=-0.135 0.156 0.111 rpy=0 0 0 -> xyz=-0.135 0.156 -0.066 rpy=0 0 0; parent base_link -> chassis
- joint base_back_right_axle_joint: origin xyz=-0.135 -0.156 0.111 rpy=0 0 0 -> xyz=-0.135 -0.156 -0.066 rpy=0 0 0; parent base_link -> chassis
- joint base_front_left_axle_joint: origin xyz=0.135 0.156 0.111 rpy=0 0 0 -> xyz=0.135 0.156 -0.066 rpy=0 0 0; parent base_link -> chassis
- joint base_front_right_axle_joint: origin xyz=0.135 -0.156 0.111 rpy=0 0 0 -> xyz=0.135 -0.156 -0.066 rpy=0 0 0; parent base_link -> chassis
